File: Esquemático Elétrico/Esquemático/Projeto_Microcontroladores.kicad_sch (KiCad schematic)
At the start: 9 parts, among them J1 USB3_B_Micro, SW1 Push button

Commit message: update(esquemático): schematics correction
Parts:
- removed J1: USB3_B_Micro, symbol Connector:USB3_B_Micro
Connections:
- net +3.3V: now also R1.1, U2.1 (VCC)
- net +5V: now also U1.39 (VSYS); no longer R1.1, U2.1 (VCC), U3.1 (VCC), U4.1 (VCC), U5.1 (VH)
- net VBUS: no longer names the net of U1.40 (VBUS)
- new net +6V: U3.1 (VCC), U4.1 (VCC), U5.1 (VH)
